Commit message: moveo

File: install/moveo_description/share/moveo_description/urdf/moveo.urdf (robot description, URDF)
Before this commit: robot moveo_urdf, 13 links, 12 joints
Links:
- removed link Gripper_Idol_Gear
- removed link Gripper_Servo_Gear
- removed link Link_1
- removed link Link_2
- removed link Link_3
- removed link Link_4
- removed link Link_5
- removed link Pivot_Arm_Gripper_Idol
- removed link Pivot_Arm_Gripper_Servo
- removed link Tip_Gripper_Idol
- removed link Tip_Gripper_Servo
- removed link odom
- added link link_1, mass 1.5994; collision mesh filename=package://moveo_description/new_meshes/link_1.STL; visual mesh filename=package://moveo_description/new_meshes/link_1.STL
- added link link_2, mass 1.7861; collision mesh filename=package://moveo_description/new_meshes/link_2.STL; visual mesh filename=package://moveo_description/new_meshes/link_2.STL
- added link link_3, mass 0.65465; collision mesh filename=package://moveo_description/new_meshes/link_3.STL; visual mesh filename=package://moveo_description/new_meshes/link_3.STL
- added link link_4, mass 0.26135; collision mesh filename=package://moveo_description/new_meshes/link_4.STL; visual mesh filename=package://moveo_description/new_meshes/link_4.STL
- added link link_5, mass 0.18973; collision mesh filename=package://moveo_description/new_meshes/link_5.STL; visual mesh filename=package://moveo_description/new_meshes/link_5.STL
- link base_link: mass None -> 0.63758; geometry collision mesh filename=package://moveo_description/new_meshes/base_link.STL; visual mesh filename=package://moveo_description/new_meshes/base_link.STL
Joints:
- removed joint Gripper_Idol_Gear_Joint
- removed joint Gripper_Servo_Gear_Joint
- removed joint Joint_1
- removed joint Joint_2
- removed joint Joint_3
- removed joint Joint_4
- removed joint Joint_5
- removed joint Pivot_Arm_Gripper_Idol_Joint
- removed joint Pivot_Arm_Gripper_Servo_Joint
- removed joint Tip_Gripper_Idol_Joint
- removed joint Tip_Gripper_Servo_Joint
- removed joint odom_joint
- added joint joint_1: type revolute, parent base_link, child link_1, origin xyz=0 0 0.066 rpy=0 0 0, axis 0 0 1, limit lower=-1.57 upper=1.57 effort=10 velocity=10
- added joint joint_2: type revolute, parent link_1, child link_2, origin xyz=0 0 0.1655 rpy=0 0 0, axis 1 0 0, limit lower=-1.57 upper=1.57 effort=10 velocity=10
- added joint joint_3: type revolute, parent link_2, child link_3, origin xyz=0.001 0 0.22112 rpy=0 0 0, axis -1 0 0, limit lower=-1.57 upper=1.57 effort=10 velocity=10
- added joint joint_4: type revolute, parent link_3, child link_4, origin xyz=0 0 0.128 rpy=0 0 0, axis 0 0 1, limit lower=-1.57 upper=1.57 effort=10 velocity=10
- added joint joint_5: type revolute, parent link_4, child link_5, origin xyz=0 0 0.095 rpy=0 0 0, axis -1 0 0, limit lower=-1.57 upper=1.57 effort=10 velocity=10

Commit message: moveo

File: install/moveo_description/share/moveo_description/urdf/moveo.urdf (robot description, URDF)
Before this commit: robot moveo_description, 6 links, 5 joints
Links:
- removed link link_1
- removed link link_2
- removed link link_3
- removed link link_4
- removed link link_5
- added link link1, mass 4.09871887854989; collision mesh filename=package://moveo_description/new_meshes/link1.STL; visual mesh filename=package://moveo_description/new_meshes/link1.STL
- added link link2, mass 1.89178197363552; collision mesh filename=package://moveo_description/new_meshes/link2.STL; visual mesh filename=package://moveo_description/new_meshes/link2.STL
- added link link3, mass 0.654645131485646; collision mesh filename=package://moveo_description/new_meshes/link3.STL; visual mesh filename=package://moveo_description/new_meshes/link3.STL
- added link link4, mass 0.605543805564186; collision mesh filename=package://moveo_description/new_meshes/link4.STL; visual mesh filename=package://moveo_description/new_meshes/link4.STL
- added link link5, mass 0.190555732375089; collision mesh filename=package://moveo_description/new_meshes/link5.STL; visual mesh filename=package://moveo_description/new_meshes/link5.STL
- added link link_L_arm, mass 0.010285; collision mesh filename=package://moveo_description/new_meshes/link_L_arm.STL; visual mesh filename=package://moveo_description/new_meshes/link_L_arm.STL
- added link link_L_gear, mass 0.00490511696862488; collision mesh filename=package://moveo_description/new_meshes/link_L_gear.STL; visual mesh filename=package://moveo_description/new_meshes/link_L_gear.STL
- added link link_L_pivot, mass 0.0016375234480386; collision mesh filename=package://moveo_description/new_meshes/link_L_pivot.STL; visual mesh filename=package://moveo_description/new_meshes/link_L_pivot.STL
- added link link_R_arm, mass 0.0102853843072999; collision mesh filename=package://moveo_description/new_meshes/link_R_arm.STL; visual mesh filename=package://moveo_description/new_meshes/link_R_arm.STL
- added link link_R_gear, mass 0.00478292072521564; collision mesh filename=package://moveo_description/new_meshes/link_R_gear.STL; visual mesh filename=package://moveo_description/new_meshes/link_R_gear.STL
- added link link_R_pivot, mass 0.00163752344803857; collision mesh filename=package://moveo_description/new_meshes/link_R_pivot.STL; visual mesh filename=package://moveo_description/new_meshes/link_R_pivot.STL
- link base_link: mass 0.63758 -> 7.78538512369426
Joints:
- removed joint joint_1
- removed joint joint_2
- removed joint joint_3
- removed joint joint_4
- removed joint joint_5
- added joint joint1: type revolute, parent base_link, child link1, origin xyz=0 -0.2425 0.017144 rpy=0 0 -0.3927, axis 0 0 1, limit lower=-1.57 upper=1.57 effort=10 velocity=10
- added joint joint2: type revolute, parent link1, child link2, origin xyz=0 0 0.1655 rpy=0 0 0, axis 1 0 0, limit lower=-1.57 upper=1.57 effort=10 velocity=10
- added joint joint3: type revolute, parent link2, child link3, origin xyz=0.001 0 0.22112 rpy=0 0 0, axis -1 0 0, limit lower=-1.57 upper=1.57 effort=10 velocity=10
- added joint joint4: type revolute, parent link3, child link4, origin xyz=0 0 0.128 rpy=0 0 0, axis 0 0 -1, limit lower=-1.57 upper=1.57 effort=10 velocity=0
- added joint joint5: type revolute, parent link4, child link5, origin xyz=0 0 0.095 rpy=0 0 0, axis -1 0 0, limit lower=-1.57 upper=1.57 effort=10 velocity=10
- added joint joint_L_arm: type revolute, parent link_L_gear, child link_L_arm, origin xyz=-0.04 0 0 rpy=0 0 0, axis 0 -1 0, limit lower=0 upper=0 effort=0 velocity=0, mimic joint=joint_R_gear multiplier=1 offset=0
- added joint joint_L_gear: type revolute, parent link5, child link_L_gear, origin xyz=-0.014 0.003 0.065 rpy=0 0 0, axis 0 -1 0, limit lower=0 upper=0 effort=2 velocity=3, mimic joint=joint_R_gear multiplier=-1 offset=0
- added joint joint_L_pivot: type revolute, parent link5, child link_L_pivot, origin xyz=-0.007 0.003 0.085 rpy=0 0 0, axis 0 -1 0, limit lower=0 upper=0 effort=0 velocity=0, mimic joint=joint_R_gear multiplier=-1 offset=0
- added joint joint_R_arm: type revolute, parent link_R_gear, child link_R_arm, origin xyz=0.04 0 0 rpy=0 0 0, axis 0 -1 0, limit lower=0 upper=0 effort=0 velocity=0, mimic joint=joint_R_gear multiplier=-1 offset=0
- added joint joint_R_gear: type revolute, parent link5, child link_R_gear, origin xyz=0.014 0.003 0.065 rpy=0 0 0, axis 0 -1 0, limit lower=0 upper=1.57 effort=2 velocity=3
- added joint joint_R_pivot: type revolute, parent link5, child link_R_pivot, origin xyz=0.007 0.003 0.085 rpy=0 0 0, axis 0 -1 0, limit lower=0 upper=0 effort=0 velocity=0, mimic joint=joint_R_gear multiplier=1 offset=0

File: install/moveo_description/share/moveo_description/urdf/moveo.urdf.xacro (robot description, xacro)
@@ -1,19 +1,20 @@
 <?xml version="1.0" encoding="utf-8"?>
-<robot xmlns:xacro="https://www.ros.org/wiki/xacro" name="moveo_description">
+<robot
+  name="moveo_description" xmlns:xacro="https://www.ros.org/wiki/xacro">
   <link
     name="base_link">
     <inertial>
       <origin
-        xyz="1.4509E-05 1.4418E-08 0.037157"
-        rpy="0 0 0" />
-      <mass
-        value="0.63758" />
-      <inertia
-        ixx="0.0015156"
-        ixy="-4.4377E-10"
-        ixz="-1.5691E-07"
-        iyy="0.0015149"
-        iyz="-1.9031E-11"
-        izz="0.0026238" />
+        xyz="0.0365462732079447 -0.0506188103426008 0.199844889715612"
+        rpy="0 0 0" />
+      <mass
+        value="7.78538512369426" />
+      <inertia
+        ixx="0.125809436671389"
+        ixy="-2.17154321475808E-05"
+        ixz="-0.000710135774901524"
+        iyy="0.250362455885131"
+        iyz="-2.98996010937198E-05"
+        izz="0.127310826437195" />
     </inertial>
     <visual>
@@ -28,5 +29,5 @@
         name="">
         <color
-          rgba="0.79216 0.81961 0.93333 1" />
+          rgba="0.784313725490196 0.784313725490196 0.784313725490196 1" />
       </material>
     </visual>
@@ -42,53 +43,53 @@
   </link>
   <link
-    name="link_1">
-    <inertial>
-      <origin
-        xyz="-9.1738E-05 -1.2493E-05 0.083097"
-        rpy="0 0 0" />
-      <mass
-        value="1.5994" />
-      <inertia
-        ixx="0.0068504"
-        ixy="1.2404E-07"
-        ixz="3.9315E-07"
-        iyy="0.0083964"
-        iyz="-3.7032E-07"
-        izz="0.0063085" />
-    </inertial>
-    <visual>
-      <origin
-        xyz="0 0 0"
-        rpy="0 0 0" />
-      <geometry>
-        <mesh
-          filename="package://moveo_description/new_meshes/link_1.STL" />
-      </geometry>
-      <material
-        name="">
-        <color
-          rgba="0.027451 0.27059 1 1" />
-      </material>
-    </visual>
-    <collision>
-      <origin
-        xyz="0 0 0"
-        rpy="0 0 0" />
-      <geometry>
-        <mesh
-          filename="package://moveo_description/new_meshes/link_1.STL" />
-      </geometry>
-    </collision>
-  </link>
-  <joint
-    name="joint_1"
-    type="revolute">
-    <origin
-      xyz="0 0 0.066"
-      rpy="0 0 0" />
+    name="link1">
+    <inertial>
+      <origin
+        xyz="-3.57977936522591E-05 -4.87510083063691E-06 0.0712687687792384"
+        rpy="0 0 0" />
+      <mass
+        value="4.09871887854989" />
+      <inertia
+        ixx="0.00799058297785298"
+        ixy="1.24041065267073E-07"
+        ixz="3.93151290964323E-07"
+        iyy="0.00908418285615879"
+        iyz="-3.70320127565607E-07"
+        izz="0.006994499363074" />
+    </inertial>
+    <visual>
+      <origin
+        xyz="0 0 0"
+        rpy="0 0 0" />
+      <geometry>
+        <mesh
+          filename="package://moveo_description/new_meshes/link1.STL" />
+      </geometry>
+      <material
+        name="">
+        <color
+          rgba="1.0 0.647 0.0 1" />
+      </material>
+    </visual>
+    <collision>
+      <origin
+        xyz="0 0 0"
+        rpy="0 0 0" />
+      <geometry>
+        <mesh
+          filename="package://moveo_description/new_meshes/link1.STL" />
+      </geometry>
+    </collision>
+  </link>
+  <joint
+    name="joint1"
+    type="revolute">
+    <origin
+      xyz="0 -0.2425 0.017144"
+      rpy="0 0 -0.3927" />
     <parent
       link="base_link" />
     <child
-      link="link_1" />
+      link="link1" />
     <axis
       xyz="0 0 1" />
@@ -100,45 +101,45 @@
   </joint>
   <link
-    name="link_2">
-    <inertial>
-      <origin
-        xyz="-0.00044845 -2.0917E-05 0.075983"
-        rpy="0 0 0" />
-      <mass
-        value="1.7861" />
-      <inertia
-        ixx="0.0048246"
-        ixy="-1.0807E-06"
-        ixz="-9.752E-06"
-        iyy="0.0049236"
-        iyz="1.8268E-07"
-        izz="0.002844" />
-    </inertial>
-    <visual>
-      <origin
-        xyz="0 0 0"
-        rpy="0 0 0" />
-      <geometry>
-        <mesh
-          filename="package://moveo_description/new_meshes/link_2.STL" />
-      </geometry>
-      <material
-        name="">
-        <color
-          rgba="0.75294 0.75294 0.75294 1" />
-      </material>
-    </visual>
-    <collision>
-      <origin
-        xyz="0 0 0"
-        rpy="0 0 0" />
-      <geometry>
-        <mesh
-          filename="package://moveo_description/new_meshes/link_2.STL" />
-      </geometry>
-    </collision>
-  </link>
-  <joint
-    name="joint_2"
+    name="link2">
+    <inertial>
+      <origin
+        xyz="-0.00181996389784646 -1.98912195225331E-05 0.0778007474155114"
+        rpy="0 0 0" />
+      <mass
+        value="1.89178197363552" />
+      <inertia
+        ixx="0.00484970489758287"
+        ixy="-1.0695114087409E-06"
+        ixz="-9.71369731067025E-06"
+        iyy="0.00497261074755014"
+        iyz="1.83373459594234E-07"
+        izz="0.00289299349274461" />
+    </inertial>
+    <visual>
+      <origin
+        xyz="0 0 0"
+        rpy="0 0 0" />
+      <geometry>
+        <mesh
+          filename="package://moveo_description/new_meshes/link2.STL" />
+      </geometry>
+      <material
+        name="">
+        <color
+          rgba="1.0 0.647 0.0 1" />
+      </material>
+    </visual>
+    <collision>
+      <origin
+        xyz="0 0 0"
+        rpy="0 0 0" />
+      <geometry>
+        <mesh
+          filename="package://moveo_description/new_meshes/link2.STL" />
+      </geometry>
+    </collision>
+  </link>
+  <joint
+    name="joint2"
     type="revolute">
     <origin
@@ -146,7 +147,7 @@
       rpy="0 0 0" />
     <parent
-      link="link_1" />
-    <child
-      link="link_2" />
+      link="link1" />
+    <child
+      link="link2" />
     <axis
       xyz="1 0 0" />
@@ -158,45 +159,45 @@
   </joint>
   <link
-    name="link_3">
-    <inertial>
-      <origin
-        xyz="-0.00035774 -8.5304E-05 0.037984"
-        rpy="0 0 0" />
-      <mass
-        value="0.65465" />
-      <inertia
-        ixx="0.0019581"
-        ixy="-5.4089E-09"
-        ixz="2.1501E-06"
-        iyy="0.0016825"
-        iyz="-5.977E-07"
-        izz="0.00042425" />
-    </inertial>
-    <visual>
-      <origin
-        xyz="0 0 0"
-        rpy="0 0 0" />
-      <geometry>
-        <mesh
-          filename="package://moveo_description/new_meshes/link_3.STL" />
-      </geometry>
-      <material
-        name="">
-        <color
-          rgba="1 1 1 1" />
-      </material>
-    </visual>
-    <collision>
-      <origin
-        xyz="0 0 0"
-        rpy="0 0 0" />
-      <geometry>
-        <mesh
-          filename="package://moveo_description/new_meshes/link_3.STL" />
-      </geometry>
-    </collision>
-  </link>
-  <joint
-    name="joint_3"
+    name="link3">
+    <inertial>
+      <origin
+        xyz="-0.000357737800626479 -8.53039392533228E-05 0.037983876263002"
+        rpy="0 0 0" />
+      <mass
+        value="0.654645131485646" />
+      <inertia
+        ixx="0.00195809921094727"
+        ixy="-5.40892730724243E-09"
+        ixz="2.15013852904307E-06"
+        iyy="0.001682518955775"
+        iyz="-5.97702340707974E-07"
+        izz="0.000424251954161472" />
+    </inertial>
+    <visual>
+      <origin
+        xyz="0 0 0"
+        rpy="0 0 0" />
+      <geometry>
+        <mesh
+          filename="package://moveo_description/new_meshes/link3.STL" />
+      </geometry>
+      <material
+        name="">
+        <color
+          rgba="1.0 0.647 0.0 1" />
+      </material>
+    </visual>
+    <collision>
+      <origin
+        xyz="0 0 0"
+        rpy="0 0 0" />
+      <geometry>
+        <mesh
+          filename="package://moveo_description/new_meshes/link3.STL" />
+      </geometry>
+    </collision>
+  </link>
+  <joint
+    name="joint3"
     type="revolute">
     <origin
@@ -204,7 +205,7 @@
       rpy="0 0 0" />
     <parent
-      link="link_2" />
-    <child
-      link="link_3" />
+      link="link2" />
+    <child
+      link="link3" />
     <axis
       xyz="-1 0 0" />
@@ -216,45 +217,45 @@
   </joint>
   <link
-    name="link_4">
-    <inertial>
-      <origin
-        xyz="-4.4474E-05 0.00088881 0.051737"
-        rpy="0 0 0" />
-      <mass
-        value="0.26135" />
-      <inertia
-        ixx="0.00050576"
-        ixy="1.9078E-07"
-        ixz="6.4065E-07"
-        iyy="0.00059141"
-        iyz="9.8116E-06"
-        izz="0.00028852" />
-    </inertial>
-    <visual>
-      <origin
-        xyz="0 0 0"
-        rpy="0 0 0" />
-      <geometry>
-        <mesh
-          filename="package://moveo_description/new_meshes/link_4.STL" />
-      </geometry>
-      <material
-        name="">
-        <color
-          rgba="0.29412 0.29412 0.29412 1" />
-      </material>
-    </visual>
-    <collision>
-      <origin
-        xyz="0 0 0"
-        rpy="0 0 0" />
-      <geometry>
-        <mesh
-          filename="package://moveo_description/new_meshes/link_4.STL" />
-      </geometry>
-    </collision>
-  </link>
-  <joint
-    name="joint_4"
+    name="link4">
+    <inertial>
+      <origin
+        xyz="-0.0122132917992238 0.000384668649412917 0.0437300556678256"
+        rpy="0 0 0" />
+      <mass
+        value="0.605543805564186" />
+      <inertia
+        ixx="0.000571210604293686"
+        ixy="1.9076448362183E-07"
+        ixz="6.40654290847272E-07"
+        iyy="0.000663775745262407"
+        iyz="9.81158210207296E-06"
+        izz="0.00036088010327795" />
+    </inertial>
+    <visual>
+      <origin
+        xyz="0 0 0"
+        rpy="0 0 0" />
+      <geometry>
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