Commit message: moveo

File: install/moveo_description/share/moveo_description/urdf/moveo.urdf (robot description, URDF)
Before this commit: robot moveo_description, 12 links, 11 joints
Links:
- link base_link: geometry collision mesh filename=package://moveo_description/meshes/base_link.STL; visual mesh filename=package://moveo_description/meshes/base_link.STL
- link link1: geometry collision mesh filename=package://moveo_description/meshes/link1.STL; visual mesh filename=package://moveo_description/meshes/link1.STL
- link link2: geometry collision mesh filename=package://moveo_description/meshes/link2.STL; visual mesh filename=package://moveo_description/meshes/link2.STL
- link link3: geometry collision mesh filename=package://moveo_description/meshes/link3.STL; visual mesh filename=package://moveo_description/meshes/link3.STL
- link link4: geometry collision mesh filename=package://moveo_description/meshes/link4.STL; visual mesh filename=package://moveo_description/meshes/link4.STL
- link link5: geometry collision mesh filename=package://moveo_description/meshes/link5.STL; visual mesh filename=package://moveo_description/meshes/link5.STL
- link link_L_arm: geometry collision mesh filename=package://moveo_description/meshes/link_L_arm.STL; visual mesh filename=package://moveo_description/meshes/link_L_arm.STL
- link link_L_gear: geometry collision mesh filename=package://moveo_description/meshes/link_L_gear.STL; visual mesh filename=package://moveo_description/meshes/link_L_gear.STL
- link link_L_pivot: geometry collision mesh filename=package://moveo_description/meshes/link_L_pivot.STL; visual mesh filename=package://moveo_description/meshes/link_L_pivot.STL
- link link_R_arm: geometry collision mesh filename=package://moveo_description/meshes/link_R_arm.STL; visual mesh filename=package://moveo_description/meshes/link_R_arm.STL
- link link_R_gear: geometry collision mesh filename=package://moveo_description/meshes/link_R_gear.STL; visual mesh filename=package://moveo_description/meshes/link_R_gear.STL
- link link_R_pivot: geometry collision mesh filename=package://moveo_description/meshes/link_R_pivot.STL; visual mesh filename=package://moveo_description/meshes/link_R_pivot.STL

File: install/moveo_description/share/moveo_description/urdf/moveo.urdf.xacro (robot description, xacro)
@@ -24,5 +24,5 @@
       <geometry>
         <mesh
-          filename="package://moveo_description/new_meshes/base_link.STL" />
+          filename="package://moveo_description/meshes/base_link.STL" />
       </geometry>
       <material
@@ -38,5 +38,5 @@
       <geometry>
         <mesh
-          filename="package://moveo_description/new_meshes/base_link.STL" />
+          filename="package://moveo_description/meshes/base_link.STL" />
       </geometry>
     </collision>
@@ -64,5 +64,5 @@
       <geometry>
         <mesh
-          filename="package://moveo_description/new_meshes/link1.STL" />
+          filename="package://moveo_description/meshes/link1.STL" />
       </geometry>
       <material
@@ -78,5 +78,5 @@
       <geometry>
         <mesh
-          filename="package://moveo_description/new_meshes/link1.STL" />
+          filename="package://moveo_description/meshes/link1.STL" />
       </geometry>
     </collision>
@@ -122,5 +122,5 @@
       <geometry>
         <mesh
-          filename="package://moveo_description/new_meshes/link2.STL" />
+          filename="package://moveo_description/meshes/link2.STL" />
       </geometry>
       <material
@@ -136,5 +136,5 @@
       <geometry>
         <mesh
-          filename="package://moveo_description/new_meshes/link2.STL" />
+          filename="package://moveo_description/meshes/link2.STL" />
       </geometry>
     </collision>
@@ -180,5 +180,5 @@
       <geometry>
         <mesh
-          filename="package://moveo_description/new_meshes/link3.STL" />
+          filename="package://moveo_description/meshes/link3.STL" />
       </geometry>
       <material
@@ -194,5 +194,5 @@
       <geometry>
         <mesh
-          filename="package://moveo_description/new_meshes/link3.STL" />
+          filename="package://moveo_description/meshes/link3.STL" />
       </geometry>
     </collision>
@@ -238,5 +238,5 @@
       <geometry>
         <mesh
-          filename="package://moveo_description/new_meshes/link4.STL" />
+          filename="package://moveo_description/meshes/link4.STL" />
       </geometry>
       <material
@@ -252,5 +252,5 @@
       <geometry>
         <mesh
-          filename="package://moveo_description/new_meshes/link4.STL" />
+          filename="package://moveo_description/meshes/link4.STL" />
       </geometry>
     </collision>
@@ -296,5 +296,5 @@
       <geometry>
         <mesh
-          filename="package://moveo_description/new_meshes/link5.STL" />
+          filename="package://moveo_description/meshes/link5.STL" />
       </geometry>
       <material
@@ -310,5 +310,5 @@
       <geometry>
         <mesh
-          filename="package://moveo_description/new_meshes/link5.STL" />
+          filename="package://moveo_description/meshes/link5.STL" />
       </geometry>
     </collision>
@@ -354,5 +354,5 @@
       <geometry>
         <mesh
-          filename="package://moveo_description/new_meshes/link_L_gear.STL" />
+          filename="package://moveo_description/meshes/link_L_gear.STL" />
       </geometry>
       <material
@@ -368,5 +368,5 @@
       <geometry>
         <mesh
-          filename="package://moveo_description/new_meshes/link_L_gear.STL" />
+          filename="package://moveo_description/meshes/link_L_gear.STL" />
       </geometry>
     </collision>
@@ -416,5 +416,5 @@
       <geometry>
         <mesh
-          filename="package://moveo_description/new_meshes/link_L_arm.STL" />
+          filename="package://moveo_description/meshes/link_L_arm.STL" />
       </geometry>
       <material
@@ -430,5 +430,5 @@
       <geometry>
         <mesh
-          filename="package://moveo_description/new_meshes/link_L_arm.STL" />
+          filename="package://moveo_description/meshes/link_L_arm.STL" />
       </geometry>
     </collision>
@@ -478,5 +478,5 @@
       <geometry>
         <mesh
-          filename="package://moveo_description/new_meshes/link_R_gear.STL" />
+          filename="package://moveo_description/meshes/link_R_gear.STL" />
       </geometry>
       <material
@@ -492,5 +492,5 @@
       <geometry>
         <mesh
-          filename="package://moveo_description/new_meshes/link_R_gear.STL" />
+          filename="package://moveo_description/meshes/link_R_gear.STL" />
       </geometry>
     </collision>
@@ -536,5 +536,5 @@
       <geometry>
         <mesh
-          filename="package://moveo_description/new_meshes/link_R_arm.STL" />
+          filename="package://moveo_description/meshes/link_R_arm.STL" />
       </geometry>
       <material
@@ -550,5 +550,5 @@
       <geometry>
         <mesh
-          filename="package://moveo_description/new_meshes/link_R_arm.STL" />
+          filename="package://moveo_description/meshes/link_R_arm.STL" />
       </geometry>
     </collision>
@@ -598,5 +598,5 @@
       <geometry>
         <mesh
-          filename="package://moveo_description/new_meshes/link_L_pivot.STL" />
+          filename="package://moveo_description/meshes/link_L_pivot.STL" />
       </geometry>
       <material
@@ -612,5 +612,5 @@
       <geometry>
         <mesh
-          filename="package://moveo_description/new_meshes/link_L_pivot.STL" />
+          filename="package://moveo_description/meshes/link_L_pivot.STL" />
       </geometry>
     </collision>
@@ -660,5 +660,5 @@
       <geometry>
         <mesh
-          filename="package://moveo_description/new_meshes/link_R_pivot.STL" />
+          filename="package://moveo_description/meshes/link_R_pivot.STL" />
       </geometry>
       <material
@@ -674,5 +674,5 @@
       <geometry>
         <mesh
-          filename="package://moveo_description/new_meshes/link_R_pivot.STL" />
+          filename="package://moveo_description/meshes/link_R_pivot.STL" />
       </geometry>
     </collision>
