Commit message: moveo

File: install/moveo_description/share/moveo_description/urdf/gazebo.urdf.xacro (robot description, xacro)
@@ -1,10 +1,24 @@
-<?xml version='1.0'?>
-<robot xmlns:xacro="https://www.ros.org/wiki/xacro" name="moveo_description">
-  <!-- <link name="World"/> -->
+<?xml version="1.0" encoding="utf-8"?>
+<robot
+  name="moveo_description" xmlns:xacro="https://www.ros.org/wiki/xacro">
   <link
     name="base_link">
-    <visual>
-      <origin
-        xyz="0 0 .13"
+    <inertial>
+      <origin
+        xyz="0.0365462732079447 -0.0506188103426008 0.199844889715612"
+        rpy="0 0 0" />
+      <mass
+        value="7.78538512369426" />
+      <inertia
+        ixx="0.125809436671389"
+        ixy="-2.17154321475808E-05"
+        ixz="-0.000710135774901524"
+        iyy="0.250362455885131"
+        iyz="-2.98996010937198E-05"
+        izz="0.127310826437195" />
+    </inertial>
+    <visual>
+      <origin
+        xyz="0 0 0"
         rpy="0 0 0" />
       <geometry>
@@ -15,713 +29,674 @@
         name="">
         <color
-          rgba="0.75294 0.75294 0.75294 1" />
-      </material>
-    </visual>
-    <collision>
-      <origin
-        xyz="0 0 .13"
-        rpy="0 0 0" />
-      <geometry>
-        <mesh
-          filename="package://moveo_description/meshes/base_link_col.STL" />
-      </geometry>
-    </collision>
-  </link>
-  <!-- dummy link -->
-  <link
-    name="odom">
-    <inertial>
-      <origin
-        xyz="0.034155 -0.20591 -0.049641"
-        rpy="0 0 0" />
-      <mass
-        value="8.0643" />
-      <inertia
-        ixx="0.11291"
-        ixy="0.00066071"
-        ixz="-0.00030472"
-        iyy="0.089946"
-        iyz="0.011461"
-        izz="0.19187" />
-    </inertial>
-   </link>
-  <joint
-    name="odom_joint"
-    type="fixed">
-    <origin
-      xyz="0 0 0"
-      rpy="0 0 0" />
+          rgba="0.784313725490196 0.784313725490196 0.784313725490196 1" />
+      </material>
+    </visual>
+    <collision>
+      <origin
+        xyz="0 0 0"
+        rpy="0 0 0" />
+      <geometry>
+        <mesh
+          filename="package://moveo_description/meshes/base_link.STL" />
+      </geometry>
+    </collision>
+  </link>
+  <link
+    name="link1">
+    <inertial>
+      <origin
+        xyz="-3.57977936522591E-05 -4.87510083063691E-06 0.0712687687792384"
+        rpy="0 0 0" />
+      <mass
+        value="4.09871887854989" />
+      <inertia
+        ixx="0.00799058297785298"
+        ixy="1.24041065267073E-07"
+        ixz="3.93151290964323E-07"
+        iyy="0.00908418285615879"
+        iyz="-3.70320127565607E-07"
+        izz="0.006994499363074" />
+    </inertial>
+    <visual>
+      <origin
+        xyz="0 0 0"
+        rpy="0 0 0" />
+      <geometry>
+        <mesh
+          filename="package://moveo_description/meshes/link1.STL" />
+      </geometry>
+      <material
+        name="">
+        <color
+          rgba="1.0 0.647 0.0 1" />
+      </material>
+    </visual>
+    <collision>
+      <origin
+        xyz="0 0 0"
+        rpy="0 0 0" />
+      <geometry>
+        <mesh
+          filename="package://moveo_description/meshes/link1.STL" />
+      </geometry>
+    </collision>
+  </link>
+  <joint
+    name="joint1"
+    type="revolute">
+    <origin
+      xyz="0 -0.2425 0.017144"
+      rpy="0 0 -0.3927" />
     <parent
       link="base_link" />
     <child
-      link="odom" />
-  </joint>
-  <link
-    name="Link_1">
-    <inertial>
-      <origin
-        xyz="4.0186E-05 0.090634 0.00010221"
-        rpy="0 0 0" />
-      <mass
-        value="4.2526" />
-      <inertia
-        ixx="0.0034071"
-        ixy="8.9041E-06"
-        ixz="1.179E-07"
-        iyy="0.018642"
-        iyz="-3.6544E-06"
-        izz="0.021987" />
-    </inertial>
-    <visual>
-      <origin
-        xyz="0 0 0"
-        rpy="0 0 0" />
-      <geometry>
-        <mesh
-          filename="package://moveo_description/meshes/Link_1.STL" />
-      </geometry>
-      <material
-        name="">
-        <color
-          rgba="0.75294 0.75294 0.75294 1" />
-      </material>
-    </visual>
-    <collision>
-      <origin
-        xyz="0 0 0"
-        rpy="0 0 0" />
-      <geometry>
-        <mesh
-          filename="package://moveo_description/meshes/Link_1_col.STL" />
-      </geometry>
-    </collision>
-  </link>
-  <joint
-    name="Joint_1"
-    type="revolute">
-    <origin
-      xyz="0 -0.2425 .13"
-      rpy="1.5708 9.5417E-17 2.7766" />
-    <parent
-      link="base_link" />
-    <child
-      link="Link_1" />
-    <axis
-      xyz="0 1 0" />
-    <limit
-      lower="-1.5707"
-      upper="1.5707"
-      effort="5"
-      velocity="1" />
-  </joint>
-  <link
-    name="Link_2">
-    <inertial>
-      <origin
-        xyz="2.2815E-05 0.0017616 -0.080002"
-        rpy="0 0 0" />
-      <mass
-        value="1.9323" />
-      <inertia
-        ixx="0.012138"
-        ixy="-3.5576E-06"
-        ixz="-9.0632E-06"
-        iyy="0.011445"
-        iyz="0.00014273"
-        izz="0.00070271" />
-    </inertial>
-    <visual>
-      <origin
-        xyz="0 0 0"
-        rpy="0 0 0" />
-      <geometry>
-        <mesh
-          filename="package://moveo_description/meshes/Link_2.STL" />
-      </geometry>
-      <material
-        name="">
-        <color
-          rgba="0.75294 0.75294 0.75294 1" />
-      </material>
-    </visual>
-    <collision>
-      <origin
-        xyz="0 0 0"
-        rpy="0 0 0" />
-      <geometry>
-        <mesh
-          filename="package://moveo_description/meshes/Link_2_col.STL" />
-      </geometry>
-    </collision>
-  </link>
-  <joint
-    name="Joint_2"
-    type="revolute">
-    <origin
-      xyz="0 0.18264 0"
-      rpy="-3.1416 0.95134 1.5708" />
-    <parent
-      link="Link_1" />
-    <child
-      link="Link_2" />
+      link="link1" />
+    <axis
+      xyz="0 0 1" />
+    <limit
+      lower="-1.57"
+      upper="1.57"
+      effort="10"
+      velocity="10" />
+  </joint>
+  <link
+    name="link2">
+    <inertial>
+      <origin
+        xyz="-0.00181996389784646 -1.98912195225331E-05 0.0778007474155114"
+        rpy="0 0 0" />
+      <mass
+        value="1.89178197363552" />
+      <inertia
+        ixx="0.00484970489758287"
+        ixy="-1.0695114087409E-06"
+        ixz="-9.71369731067025E-06"
+        iyy="0.00497261074755014"
+        iyz="1.83373459594234E-07"
+        izz="0.00289299349274461" />
+    </inertial>
+    <visual>
+      <origin
+        xyz="0 0 0"
+        rpy="0 0 0" />
+      <geometry>
+        <mesh
+          filename="package://moveo_description/meshes/link2.STL" />
+      </geometry>
+      <material
+        name="">
+        <color
+          rgba="1.0 0.647 0.0 1" />
+      </material>
+    </visual>
+    <collision>
+      <origin
+        xyz="0 0 0"
+        rpy="0 0 0" />
+      <geometry>
+        <mesh
+          filename="package://moveo_description/meshes/link2.STL" />
+      </geometry>
+    </collision>
+  </link>
+  <joint
+    name="joint2"
+    type="revolute">
+    <origin
+      xyz="0 0 0.1655"
+      rpy="0 0 0" />
+    <parent
+      link="link1" />
+    <child
+      link="link2" />
+    <axis
+      xyz="1 0 0" />
+    <limit
+      lower="-1.57"
+      upper="1.57"
+      effort="10"
+      velocity="10" />
+  </joint>
+  <link
+    name="link3">
+    <inertial>
+      <origin
+        xyz="-0.000357737800626479 -8.53039392533228E-05 0.037983876263002"
+        rpy="0 0 0" />
+      <mass
+        value="0.654645131485646" />
+      <inertia
+        ixx="0.00195809921094727"
+        ixy="-5.40892730724243E-09"
+        ixz="2.15013852904307E-06"
+        iyy="0.001682518955775"
+        iyz="-5.97702340707974E-07"
+        izz="0.000424251954161472" />
+    </inertial>
+    <visual>
+      <origin
+        xyz="0 0 0"
+        rpy="0 0 0" />
+      <geometry>
+        <mesh
+          filename="package://moveo_description/meshes/link3.STL" />
+      </geometry>
+      <material
+        name="">
+        <color
+          rgba="1.0 0.647 0.0 1" />
+      </material>
+    </visual>
+    <collision>
+      <origin
+        xyz="0 0 0"
+        rpy="0 0 0" />
+      <geometry>
+        <mesh
+          filename="package://moveo_description/meshes/link3.STL" />
+      </geometry>
+    </collision>
+  </link>
+  <joint
+    name="joint3"
+    type="revolute">
+    <origin
+      xyz="0.001 0 0.22112"
+      rpy="0 0 0" />
+    <parent
+      link="link2" />
+    <child
+      link="link3" />
+    <axis
+      xyz="-1 0 0" />
+    <limit
+      lower="-1.57"
+      upper="1.57"
+      effort="10"
+      velocity="10" />
+  </joint>
+  <link
+    name="link4">
+    <inertial>
+      <origin
+        xyz="-0.0122132917992238 0.000384668649412917 0.0437300556678256"
+        rpy="0 0 0" />
+      <mass
+        value="0.605543805564186" />
+      <inertia
+        ixx="0.000571210604293686"
+        ixy="1.9076448362183E-07"
+        ixz="6.40654290847272E-07"
+        iyy="0.000663775745262407"
+        iyz="9.81158210207296E-06"
+        izz="0.00036088010327795" />
+    </inertial>
+    <visual>
+      <origin
+        xyz="0 0 0"
+        rpy="0 0 0" />
+      <geometry>
+        <mesh
+          filename="package://moveo_description/meshes/link4.STL" />
+      </geometry>
+      <material
+        name="">
+        <color
+          rgba="1.0 0.647 0.0 1" />
+      </material>
+    </visual>
+    <collision>
+      <origin
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