Commit message: moveo

File: src/moveo_description/urdf/moveo.urdf (robot description, URDF)
Before this commit: robot moveo_description, 12 links, 11 joints
Joints:
- joint joint4: axis 0 0 -1 -> 0 0 1
- joint joint_L_arm: limit lower=0 upper=0 effort=0 velocity=0 -> lower=0 upper=1.57 effort=2 velocity=3
- joint joint_L_gear: limit lower=0 upper=0 effort=2 velocity=3 -> lower=-1.57 upper=0 effort=2 velocity=3
- joint joint_L_pivot: limit lower=0 upper=0 effort=0 velocity=0 -> lower=-1.57 upper=0 effort=2 velocity=3
- joint joint_R_arm: limit lower=0 upper=0 effort=0 velocity=0 -> lower=-1.57 upper=0 effort=2 velocity=3
- joint joint_R_pivot: limit lower=0 upper=0 effort=0 velocity=0 -> lower=0 upper=1.57 effort=2 velocity=3

File: src/moveo_description/urdf/moveo.urdf.xacro (robot description, xacro)
@@ -271,5 +271,5 @@
       upper="1.57"
       effort="10"
-      velocity="0" />
+      velocity="10" />
   </joint>
   <link

File: src/moveo_description/urdf/moveo_ros2_control.xacro (robot description, xacro)
@@ -30,5 +30,5 @@
             <command_interface name="position">
                 <param name="min">-${PI/2}</param>
-                <param name="max">0.0</param>
+                <param name="max">${PI/2}</param>
             </command_interface>
             <state_interface name="position"/>
@@ -43,6 +43,8 @@
         <joint name="joint_R_gear">
             <command_interface name="position">
-                <param name="min">-${PI/2}</param>
-                <param name="max">0.0</param>
+                <!-- <param name="min">-${PI/2}</param>
+                <param name="max">0.0</param> -->
+                <param name="min">0</param>
+                <param name="max">${PI/2}</param>
             </command_interface>
             <state_interface name="position"/>
